File: stm32wb_base.kicad_sch (KiCad schematic)
At the start: 60 parts, among them J1 Conn_Coaxial, J2 Conn_01x04, J3 USB_C_Receptacle_USB2.0_16P, J4 Conn_01x03, SW1 SW_Push, U1 STM32WB55CEUx, U2 USBLC6-2SC6, U3 LSM6DSO, U4 BQ24074RGT, U5 MCP16311x-xMNY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

Commit message: update company and version
Other:
- company: Overbearing Bear -> SL
Changed lines of the file:
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@@
 		(title "STM32 Basic Breakout w/ RF")
 		(date "2024-11-05")
-		(rev "V1")
-		(company "Overbearing Bear")
+		(rev "V0")
+		(company "SL")
 	)
 	(junction
